File: sensors_network/hardware/eagle/node/AA_Type/m328p_rfm69_node.brd (EAGLE design)
At the start: 65.5 x 41.7 mm, 37 parts, among them IC2 L6920, SW2 Node ID, U1 M328P, U2 RFM69W, Y1 8MHz

Commit message: final pcb's refactorings
Other:
- board text added: "Rev 1.3"
Changed lines of the file:
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@@
 <text x="35.306" y="6.096" size="1.27" layer="22" rot="MR0">AA Type</text>
 <text x="35.814" y="34.544" size="1.27" layer="22" rot="MR0">AA Type</text>
+<text x="53.848" y="1.016" size="1.27" layer="21">Rev 1.3</text>
 </plain>
 <attributes>
