File: sensors_network/hardware/eagle/node/AA_Type/m328p_rfm69_node.sch (EAGLE design)
At the start: 37 parts, among them IC2 L6920, SW2 Node ID, U1 M328P, U2 RFM69W, Y1 8MHz

Commit message: final pcb's refactorings
Other:
- note added: "Rev 1.3"
Changed lines of the file:
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@@
 <setting verticaltext="up"/>
 </settings>
-<grid distance="0.01" unitdist="inch" unit="inch" style="dots" multiple="1" display="yes" altdistance="0.01" altunitdist="inch" altunit="inch"/>
+<grid distance="0.01" unitdist="inch" unit="inch" style="lines" multiple="1" display="no" altdistance="0.01" altunitdist="inch" altunit="inch"/>
 <layers>
 <layer number="1" name="Top" color="4" fill="1" visible="no" active="no"/>
@@
 <wire x1="130.048" y1="134.874" x2="130.048" y2="85.852" width="0.1016" layer="94"/>
 <text x="134.874" y="88.9" size="1.778" layer="94" rot="R90">Node activity LED</text>
+<text x="247.142" y="5.08" size="1.778" layer="94">Rev 1.3</text>
 </plain>
 <instances>
